Commit message: (co planning motion nhung gazebo bi sap do velocity track)

File: src/so101_ros2/so101_description/urdf/so101_macro.urdf.xacro (robot description, xacro)
@@ -1,7 +1,5 @@
 <?xml version="1.0"?>
 <robot xmlns:xacro="http://www.ros.org/wiki/xacro">
-    <!-- Khai báo macro với 3 tham số: prefix, parent và khối origin -->
     <xacro:macro name="so101_arm" params="prefix parent *origin">
-        <!-- THÊM LẠI LINK ROOT Ở ĐÂY -->
         <link name="${prefix}root" />
         <link name="${prefix}base_link">
@@ -173,4 +171,5 @@
             </collision>
         </link>
+        <!-- Đã sửa số nguyên 1 thành 1.0 -->
         <joint name="${prefix}end_effector" type="revolute">
             <origin xyz="-0.018946 -0.0266092 -0.00724663" rpy="3.14159 1.29034 3.14159" />
@@ -178,7 +177,6 @@
             <parent link="${prefix}wrist_roll_follower_so101_v1" />
             <child link="${prefix}moving_jaw_so101_v1" />
-            <limit effort="1" velocity="1" lower="-1.0472" upper="1.06581e-14" />
-        </joint>
-        <!-- Khớp kết nối môi trường (world) với root của tay -->
+            <limit effort="1.0" velocity="1.0" lower="-1.0472" upper="1.06581e-14" />
+        </joint>
         <joint name="${prefix}base_mount" type="fixed">
             <xacro:insert_block name="origin" />
@@ -186,5 +184,4 @@
             <child link="${prefix}root" />
         </joint>
-        <!-- Khớp nối gốc trả lại như cũ: từ root gắn vào base_link -->
         <joint name="${prefix}fastened_1" type="fixed">
             <origin xyz="0 0 0" rpy="1.5708 0 0" />
@@ -192,4 +189,5 @@
             <child link="${prefix}base_link" />
         </joint>
+        <!-- Đã sửa số nguyên 1 thành 1.0 -->
         <joint name="${prefix}joint_1" type="revolute">
             <origin xyz="-6.93889e-18 0.031 0.05955" rpy="-1.82999e-16 -3.33067e-16 -4.74682e-17" />
@@ -197,6 +195,7 @@
             <parent link="${prefix}base_link" />
             <child link="${prefix}link_2" />
-            <limit effort="1" velocity="1" lower="-3.19407" upper="0.296587" />
-        </joint>
+            <limit effort="1.0" velocity="1.0" lower="-3.19407" upper="0.296587" />
+        </joint>
+        <!-- Đã sửa số nguyên 1 thành 1.0 -->
         <joint name="${prefix}joint_2" type="revolute">
             <origin xyz="0.0341073 0.11745 -0.0279554" rpy="-8.40441e-14 1.44874 -8.04183e-14" />
@@ -204,6 +203,7 @@
             <parent link="${prefix}link_2" />
             <child link="${prefix}link_3" />
-            <limit effort="1" velocity="1" lower="-2.64934" upper="0.492256" />
-        </joint>
+            <limit effort="1.0" velocity="1.0" lower="-2.64934" upper="0.492256" />
+        </joint>
+        <!-- Đã sửa số nguyên 1 thành 1.0 -->
         <joint name="${prefix}joint_3" type="revolute">
             <origin xyz="-5e-05 0.0917043 -0.0962012" rpy="-1.07854 1.75227e-15 4.93588e-15" />
@@ -211,6 +211,7 @@
             <parent link="${prefix}link_3" />
             <child link="${prefix}link_4" />
-            <limit effort="1" velocity="1" lower="-0.738273" upper="2.05425" />
-        </joint>
+            <limit effort="1.0" velocity="1.0" lower="-0.738273" upper="2.05425" />
+        </joint>
+        <!-- Đã sửa số nguyên 1 thành 1.0 -->
         <joint name="${prefix}joint_4" type="revolute">
             <origin xyz="-5e-05 -0.0897624 0.107881" rpy="0.657991 3.13488e-15 -1.60269e-15" />
@@ -218,5 +219,5 @@
             <parent link="${prefix}link_4" />
             <child link="${prefix}link_5" />
-            <limit effort="1" velocity="1" lower="-1.3827" upper="1.40983" />
+            <limit effort="1.0" velocity="1.0" lower="-1.3827" upper="1.40983" />
         </joint>
         <joint name="${prefix}joint_5" type="continuous">
@@ -238,5 +239,4 @@
             <child link="${prefix}mate_connector_2" />
         </joint>
-        <!-- Gắn mạch ros2_control cho từng cánh tay -->
         <ros2_control name="${prefix}System" type="system">
             <hardware>
@@ -245,30 +245,42 @@
             <joint name="${prefix}joint_1">
                 <command_interface name="position"/>
-                <state_interface name="position"/>
+                <state_interface name="position">
+                    <param name="initial_value">0.0</param>
+                </state_interface>
                 <state_interface name="velocity"/>
             </joint>
             <joint name="${prefix}joint_2">
                 <command_interface name="position"/>
-                <state_interface name="position"/>
+                <state_interface name="position">
+                    <param name="initial_value">0.0</param>
+                </state_interface>
                 <state_interface name="velocity"/>
             </joint>
             <joint name="${prefix}joint_3">
                 <command_interface name="position"/>
-                <state_interface name="position"/>
+                <state_interface name="position">
+                    <param name="initial_value">0.0</param>
+                </state_interface>
                 <state_interface name="velocity"/>
             </joint>
             <joint name="${prefix}joint_4">
                 <command_interface name="position"/>
-                <state_interface name="position"/>
+                <state_interface name="position">
+                    <param name="initial_value">0.0</param>
+                </state_interface>
                 <state_interface name="velocity"/>
             </joint>
             <joint name="${prefix}joint_5">
                 <command_interface name="position"/>
-                <state_interface name="position"/>
+                <state_interface name="position">
+                    <param name="initial_value">0.0</param>
+                </state_interface>
                 <state_interface name="velocity"/>
             </joint>
             <joint name="${prefix}end_effector">
                 <command_interface name="position"/>
-                <state_interface name="position"/>
+                <state_interface name="position">
+                    <param name="initial_value">0.0</param>
+                </state_interface>
                 <state_interface name="velocity"/>
             </joint>
